File: bridge/bridge.kicad_sch (KiCad schematic)
At the start: 6 parts, among them J101 5V, J102 5V, J103 DIN, J104 DOUT, J105 0V, J106 0V

Commit message: Update page info boxes
Other:
- title: (none) -> LEDEAF Bridge PCB
Changed lines of the file:
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@@
 (kicad_sch (version 20210406) (generator eeschema)
   (paper "A4")
+  (title_block
+    (title "LEDEAF Bridge PCB")
+    (date "2021-05-23")
+    (rev "1")
+    (comment 1 "Drawn By: AG")
+  )
   (wire (pts (xy 116.84 100.33) (xy 121.92 100.33))
     (stroke (width 0) (type solid) (color 0 0 0 0))
